Commit message: Added launch Files

File: urdf/robot.urdf.xacro (robot description, xacro)
@@ -9,4 +9,7 @@
         <box size="0.30 0.20 0.10"/>
       </geometry>
+			<material name="black">
+  			<color rgba="0 0 1 1"/>
+			</material>
     </visual>
     <collision>
@@ -21,18 +24,58 @@
     </inertial>
   </link>
-  <link name="left_wheel">
-    <visual>
-      <geometry>
-        <cylinder radius="${wheel_radius}" length="${wheel_width}"/>
-      </geometry>
-    </visual>
-  </link>
-  <link name="right_wheel">
-    <visual>
-      <geometry>
-        <cylinder radius="${wheel_radius}" length="${wheel_width}"/>
-      </geometry>
-    </visual>
-  </link>
+	<link name="left_wheel">
+		<visual>
+			<origin xyz="0 0 0" rpy="1.5707 0 0"/>
+			<geometry>
+				<cylinder radius="${wheel_radius}" length="${wheel_width}"/>
+			</geometry>
+			<material name="black">
+  			<color rgba="0 0 0 1"/>
+			</material>
+		</visual>
+		<collision>
+			<origin xyz="0 0 0" rpy="1.5707 0 0"/>
+			<geometry>
+				<cylinder radius="${wheel_radius}" length="${wheel_width}"/>
+			</geometry>
+			<material name="black">
+  			<color rgba="0 0 0 1"/>
+			</material>
+		</collision>
+		<inertial>
+			<mass value="0.2"/>
+			<origin xyz="0 0 0"/>
+			<inertia ixx="0.0005" ixy="0" ixz="0"
+							iyy="0.0005" iyz="0"
+							izz="0.0005"/>
+		</inertial>
+	</link>
+	<link name="right_wheel">
+		<visual>
+			<origin xyz="0 0 0" rpy="1.5707 0 0"/>
+			<geometry>
+				<cylinder radius="${wheel_radius}" length="${wheel_width}"/>
+			</geometry>
+			<material name="black">
+  			<color rgba="0 0 0 1"/>
+			</material>
+		</visual>
+		<collision>
+			<origin xyz="0 0 0" rpy="1.5707 0 0"/>
+			<geometry>
+				<cylinder radius="${wheel_radius}" length="${wheel_width}"/>
+			</geometry>
+			<material name="black">
+  			<color rgba="0 0 0 1"/>
+			</material>
+		</collision>
+		<inertial>
+			<mass value="0.2"/>
+			<origin xyz="0 0 0"/>
+			<inertia ixx="0.0005" ixy="0" ixz="0"
+							iyy="0.0005" iyz="0"
+							izz="0.0005"/>
+		</inertial>
+	</link>
   <link name="caster_wheel">
     <visual>
@@ -40,4 +83,7 @@
         <sphere radius="0.03"/>
       </geometry>
+			<material name="black">
+  			<color rgba="0 0 0 1"/>
+			</material>
     </visual>
   </link>
@@ -67,5 +113,5 @@
   <ros2_control name="DiffBotSystem" type="system">
     <hardware>
-      <plugin>gz_ros2_control/GazeboSimSystem</plugin>
+      <plugin>gazebo_ros2_control/GazeboSystem</plugin>
     </hardware>
     <joint name="left_wheel_joint">
@@ -80,7 +126,9 @@
     </joint>
   </ros2_control>
-  <gazebo>
-    <plugin filename="libgz_ros2_control-system.so"
-            name="gz_ros2_control::GazeboSimROS2ControlPlugin"/>
-  </gazebo>
+	<gazebo>
+		<plugin filename="libgazebo_ros2_control.so"
+						name="gazebo_ros2_control">
+			<parameters>$(find bot_controls)/config/controllers.yaml</parameters>
+		</plugin>
+	</gazebo>
 </robot>

Commit message: Added IMU Link

File: urdf/robot.urdf.xacro (robot description, xacro)
@@ -109,6 +109,19 @@
     <parent link="base_link"/>
     <child link="imu_link"/>
-    <origin xyz="0 0 0.05"/>
+    <origin xyz="0 0 0.05" rpy = "0 0 0"/>
   </joint>
+	<gazebo reference="imu_link">
+		<sensor name="imu_sensor" type="imu">
+			<always_on>true</always_on>
+			<update_rate>100</update_rate>
+			<visualize>true</visualize>
+			<plugin name="imu_plugin" filename="libgazebo_ros_imu_sensor.so">
+				<ros>
+					<namespace>/imu</namespace>
+					<remapping>~/out:=data</remapping>
+				</ros>
+			</plugin>
+		</sensor>
+	</gazebo>
   <ros2_control name="DiffBotSystem" type="system">
     <hardware>
